File: pcb/main.kicad_pcb (KiCad board)
At the start: 2 copper layers, 44.8 x 75 mm, 17 parts, among them J1 N!N, J10 Conn_01x12_Socket, J11 Conn_01x12_Socket, J2 Conn_01x12_Socket, J3 Conn_01x12_Socket, J6 Display_nice-view, J8 Conn_01x12_Socket, J9 Conn_01x12_Socket, SW37 SW_Push, SW38 RotaryEncoder_Switch

Commit message: second draft
Parts:
- removed the H1 at (59.5, 42.5)
- removed the H1 at (74.0, 111.5)
- removed the H1 at (55.5, 55.5)
- removed the H1 at (88.5, 42.5)
- added H1: MountingHole, zzkeeb:Hole_M2-solder-nut-2.5, F.Cu at (55.5, 55.5)
- added H5: MountingHole, zzkeeb:Hole_M2-solder-nut-2.5, F.Cu at (59.5, 42.5)
- added H6: MountingHole, zzkeeb:Hole_M2-solder-nut-2.5, F.Cu at (88.5, 42.5)
- added H7: MountingHole, zzkeeb:Hole_M2-solder-nut-2.5, F.Cu at (74.0, 107.0)
- added U1: RollerEncoder_EVQWGD001, zzkeeb:RotaryEncoder_EVQWGD001, F.Cu at (73.0, 97.0)
- H2, H3, H4: footprint zzkeeb:Hole_M2-TH -> zzkeeb:Hole_M2-solder-nut-2.5
- moved SW38 3.00 mm to (74.0, 97.0), turned to 180 degrees
- moved J11 1.50 mm to (92.5, 73.0)
- moved J6 1.00 mm to (74.0, 72.0)
Connections:
- J1 pad 10: row5 -> (no net)
- J1 pad 11: row6 -> (no net)
- J1 pad 12: row7 -> (no net)
- J1 pad 13: row3 -> (no net)
- J1 pad 14: row2 -> (no net)
- J1 pad 15: row1 -> (no net)
- J1 pad 16: row0 -> (no net)
- J1 pad 17: col0 -> (no net)
- J1 pad 18: col1 -> (no net)
- J1 pad 19: col2 -> (no net)
- J1 pad 2: col5 -> (no net)
- J1 pad 20: OFF -> (no net)
- J1 pad 24: BAT -> (no net)
- J1 pad 31: encA -> OFF
- J1 pad 32: encB -> (no net)
- J1 pad 33: unconnected-(J1-107-Pad33) -> (no net)
- J1 pad 7: col4 -> encA
- J1 pad 8: col3 -> encB
- J1 pad 9: row4 -> (no net)
- J10 pad 1: BAT -> (no net)
- J10 pad 10: row1 -> (no net)
- J10 pad 11: row0 -> (no net)
- J10 pad 2: col5 -> (no net)
- J10 pad 3: col4 -> (no net)
- J10 pad 4: col3 -> (no net)
- J10 pad 5: col2 -> (no net)
- J10 pad 6: col1 -> (no net)
- J10 pad 7: col0 -> (no net)
- J10 pad 8: row3 -> (no net)
- J10 pad 9: row2 -> (no net)
- J11 pad 1: BAT -> (no net)
- J11 pad 10: row1 -> (no net)
- J11 pad 11: row0 -> (no net)
- J11 pad 2: col5 -> (no net)
- J11 pad 3: col4 -> (no net)
- J11 pad 4: col3 -> (no net)
- J11 pad 5: col2 -> (no net)
- J11 pad 6: col1 -> (no net)
- J11 pad 7: col0 -> (no net)
- J11 pad 8: row3 -> (no net)
- J11 pad 9: row2 -> (no net)
- J2 pad 1: BAT -> (no net)
- J2 pad 10: row1 -> (no net)
- J2 pad 11: row0 -> (no net)
- J2 pad 12: GND -> (no net)
- J2 pad 2: col5 -> (no net)
- J2 pad 3: col4 -> (no net)
- J2 pad 4: col3 -> (no net)
- J2 pad 5: col2 -> (no net)
- J2 pad 6: col1 -> (no net)
- J2 pad 7: col0 -> GND
- J2 pad 8: row3 -> (no net)
- J2 pad 9: row2 -> (no net)
- J3 pad 1: GND -> (no net)
- J3 pad 10: col4 -> (no net)
- J3 pad 11: col5 -> (no net)
- J3 pad 12: BAT -> (no net)
- J3 pad 2: row4 -> (no net)
- J3 pad 3: row5 -> (no net)
- J3 pad 4: row6 -> (no net)
- J3 pad 5: row7 -> (no net)
- J3 pad 6: col0 -> GND
- J3 pad 7: col1 -> (no net)
- J3 pad 8: col2 -> (no net)
- J3 pad 9: col3 -> (no net)
- J8 pad 1: BAT -> (no net)
- J8 pad 10: row1 -> (no net)
- J8 pad 11: row0 -> (no net)
- J8 pad 2: col5 -> (no net)
- J8 pad 3: col4 -> (no net)
- J8 pad 4: col3 -> (no net)
- J8 pad 5: col2 -> (no net)
- J8 pad 6: col1 -> (no net)
- J8 pad 7: col0 -> (no net)
- J8 pad 8: row3 -> (no net)
- J8 pad 9: row2 -> (no net)
- J9 pad 1: BAT -> (no net)
- J9 pad 10: row1 -> (no net)
- J9 pad 11: row0 -> (no net)
- J9 pad 2: col5 -> (no net)
- J9 pad 3: col4 -> (no net)
- J9 pad 4: col3 -> (no net)
- J9 pad 5: col2 -> (no net)
- J9 pad 6: col1 -> (no net)
- J9 pad 7: col0 -> (no net)
- J9 pad 8: row3 -> (no net)
- J9 pad 9: row2 -> (no net)
Routing:
- net (no net): track 0.00 -> 775.8 mm, vias 0 -> 12
- net GND: track 120.0 -> 330.3 mm
- net row0: track 92.7 -> 0.00 mm, vias 2 -> 0
- net row1: track 79.4 -> 0.00 mm
- net col0: track 68.1 -> 0.00 mm, vias 2 -> 0
- net col1: track 66.0 -> 0.00 mm
- net col5: track 65.6 -> 0.00 mm
- net col2: track 64.4 -> 0.00 mm
- net row2: track 62.7 -> 0.00 mm
- net BAT: track 56.9 -> 0.00 mm
- net col4: track 56.1 -> 0.00 mm, vias 2 -> 0
- net row3: track 55.1 -> 0.00 mm, vias 2 -> 0
- net col3: track 54.8 -> 0.00 mm, vias 2 -> 0
- net row4: track 26.3 -> 0.00 mm
- net row5: track 22.9 -> 0.00 mm
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- removed copper zone on B.Cu, net GND
- removed copper zone on F.Cu, net GND
Other:
- board size 44.8 x 75 mm -> 44.8 x 70.5 mm
