File: pcb/connector-left.kicad_pcb (KiCad board)
At the start: 2 copper layers, 7.8 x 48.8 mm, 4 parts, among them J10 Conn_01x12_Socket, J8 Conn_01x12_Socket

Commit message: second draft
Parts:
- H1, H2: footprint zzkeeb:Hole_M2-TH -> zzkeeb:Hole_M2-solder-nut-2.5
Other:
- outline, holes or cut-outs redrawn

Commit message: add 3d components
Parts:
- H1, H2, J10: moved to B.Cu
- J8: value Conn_01x12_Socket -> C262499; moved to B.Cu
- moved H1 247.9 mm to (314.9, 101.9), turned to 90 degrees
- moved J10 227.1 mm to (297.4, 101.9), turned to 90 degrees
- moved J8 211.7 mm to (283.9, 101.9), turned to 180 degrees
- moved H2 200.7 mm to (273.9, 101.9), turned to 90 degrees
Connections:
- J10 pad 1: (no net) -> BAT-conn1
- J10 pad 10: (no net) -> row1-conn1
- J10 pad 11: (no net) -> row0-conn1
- J10 pad 12: GND -> free-conn1
- J10 pad 2: (no net) -> col4-conn1
- J10 pad 3: (no net) -> col3-conn1
- J10 pad 4: (no net) -> col2-conn1
- J10 pad 5: (no net) -> col1-conn1
- J10 pad 6: (no net) -> col0-conn1
- J10 pad 7: (no net) -> GND
- J10 pad 8: (no net) -> row3-conn1
- J10 pad 9: (no net) -> row2-conn1
- J8 pad 1: (no net) -> BAT-conn1
- J8 pad 10: (no net) -> row1-conn1
- J8 pad 11: (no net) -> row0-conn1
- J8 pad 12: GND -> free-conn1
- J8 pad 2: (no net) -> col4-conn1
- J8 pad 3: (no net) -> col3-conn1
- J8 pad 4: (no net) -> col2-conn1
- J8 pad 5: (no net) -> col1-conn1
- J8 pad 6: (no net) -> col0-conn1
- J8 pad 7: (no net) -> GND
- J8 pad 8: (no net) -> row3-conn1
- J8 pad 9: (no net) -> row2-conn1
Routing:
- net (no net): track 158.3 -> 0.00 mm, vias 5 -> 0
- net free-conn1: track 0.00 -> 24.2 mm, vias 0 -> 1
- net row0-conn1: track 0.00 -> 23.8 mm, vias 0 -> 1
- net row1-conn1: track 0.00 -> 20.9 mm
- net row2-conn1: track 0.00 -> 19.8 mm, vias 0 -> 1
- net row3-conn1: track 0.00 -> 18.0 mm, vias 0 -> 1
- net col0-conn1: track 0.00 -> 13.9 mm, vias 0 -> 1
- net col1-conn1: track 0.00 -> 13.2 mm
- net col3-conn1: track 0.00 -> 11.9 mm, vias 0 -> 1
- net col2-conn1: track 0.00 -> 10.6 mm
- net GND: track 24.1 -> 17.4 mm, vias 1 -> 0
- net col4-conn1: track 0.00 -> 6.25 mm
- net BAT-conn1: track 0.00 -> 5.75 mm
Other:
- board size 7.8 x 48.8 mm -> 48.8 x 7.8 mm
