File: pcb/pcb.kicad_pcb (KiCad board)
At the start: 2 copper layers, 206.4 x 90.7 mm, 56 parts, among them J1 N!N, J10 Conn_01x12_Socket, J11 Conn_01x12_Socket, J2 Conn_01x12_Socket, J3 Conn_01x12_Socket, J4 Conn_01x12_Socket, J5 Conn_01x12_Socket, J6 Display_nice-view, J7 Conn_01x02_Socket, J8 Conn_01x12_Socket, J9 Conn_01x12_Socket, SW1 Switch, SW10 Switch, SW11 Switch, SW12 Switch, SW13 Switch, SW14 Switch, SW15 Switch, SW16 Switch, SW17 Switch, SW18 Switch, SW2 Switch, SW3 Switch, SW37 SW_Push, SW38 RotaryEncoder_Switch, SW4 Switch, SW5 Switch, SW6 Switch, SW7 Switch, SW8 Switch, SW9 Switch

Commit message: second draft
Parts:
- added D19: D, zzkeeb:Diode_1N4148-SOD123, B.Cu at (236.2, 67.9)
- added D20: D, zzkeeb:Diode_1N4148-SOD123, B.Cu at (236.2, 60.9)
- added D21: D, zzkeeb:Diode_1N4148-SOD123, B.Cu at (233.2, 60.9)
- added D22: D, zzkeeb:Diode_1N4148-SOD123, B.Cu at (230.2, 60.9)
- added D23: D, zzkeeb:Diode_1N4148-SOD123, B.Cu at (233.2, 67.9)
- added D24: D, zzkeeb:Diode_1N4148-SOD123, B.Cu at (230.2, 93.4)
- added D25: D, zzkeeb:Diode_1N4148-SOD123, B.Cu at (236.2, 74.9)
- added D26: D, zzkeeb:Diode_1N4148-SOD123, B.Cu at (233.2, 74.9)
- added D27: D, zzkeeb:Diode_1N4148-SOD123, B.Cu at (230.2, 74.9)
- added D28: D, zzkeeb:Diode_1N4148-SOD123, B.Cu at (230.2, 67.9)
- added D29: D, zzkeeb:Diode_1N4148-SOD123, B.Cu at (236.2, 100.4)
- added D30: D, zzkeeb:Diode_1N4148-SOD123, B.Cu at (233.2, 100.4)
- added D31: D, zzkeeb:Diode_1N4148-SOD123, B.Cu at (230.2, 100.4)
- added D32: D, zzkeeb:Diode_1N4148-SOD123, B.Cu at (236.2, 93.4)
- added D33: D, zzkeeb:Diode_1N4148-SOD123, B.Cu at (233.2, 93.4)
- added D34: D, zzkeeb:Diode_1N4148-SOD123, B.Cu at (230.2, 111.4)
- added D35: D, zzkeeb:Diode_1N4148-SOD123, B.Cu at (233.2, 111.4)
- added D36: D, zzkeeb:Diode_1N4148-SOD123, B.Cu at (236.2, 111.4)
- added J12: Conn_01x02_Socket, zzkeeb:Connector_JST-1x02-2.00mm, F.Cu at (232.2, 105.4)
- added SW19: Switch, zzkeeb:Switch_MXKS-miny-hotswap-south-ks3d, F.Cu at (247.2, 65.4)
- added SW20: Switch, zzkeeb:Switch_MXKS-miny-hotswap-south-ks3d, F.Cu at (266.2, 63.4)
- added SW21: Switch, zzkeeb:Switch_MXKS-miny-hotswap-south-ks3d, F.Cu at (285.2, 57.4)
- added SW22: Switch, zzkeeb:Switch_MXKS-miny-hotswap-south-ks3d, F.Cu at (304.2, 61.4)
- added SW23: Switch, zzkeeb:Switch_MXKS-miny-hotswap-south-ks3d, F.Cu at (342.2, 83.4)
- added SW24: Switch, zzkeeb:Switch_MXKS-miny-hotswap-south-ks3d, F.Cu at (247.2, 81.4)
- added SW25: Switch, zzkeeb:Switch_MXKS-miny-hotswap-south-ks3d, F.Cu at (266.2, 79.4)
- added SW26: Switch, zzkeeb:Switch_MXKS-miny-hotswap-south-ks3d, F.Cu at (285.2, 73.4)
- added SW27: Switch, zzkeeb:Switch_MXKS-miny-hotswap-south-ks3d, F.Cu at (304.2, 77.4)
- added SW28: Switch, zzkeeb:Switch_MXKS-miny-hotswap-south-ks3d, F.Cu at (323.2, 83.4)
- added SW29: Switch, zzkeeb:Switch_MXKS-miny-hotswap-south-ks3d, F.Cu at (247.2, 97.4)
- added SW30: Switch, zzkeeb:Switch_MXKS-miny-hotswap-south-ks3d, F.Cu at (266.2, 95.4)
- added SW31: Switch, zzkeeb:Switch_MXKS-miny-hotswap-south-ks3d, F.Cu at (285.2, 89.4)
- added SW32: Switch, zzkeeb:Switch_MXKS-miny-hotswap-south-ks3d, F.Cu at (304.2, 93.4)
- added SW33: Switch, zzkeeb:Switch_MXKS-miny-hotswap-south-ks3d, F.Cu at (323.2, 99.4)
- added SW34: Switch, zzkeeb:Switch_MXKS-miny-hotswap-south-ks3d, F.Cu at (226.3, 126.4)
- added SW35: Switch, zzkeeb:Switch_MXKS-miny-hotswap-south-ks3d, F.Cu at (246.0, 121.2)
- added SW36: Switch, zzkeeb:Switch_MXKS-miny-hotswap-south-ks3d, F.Cu at (266.2, 119.4)
- added U1: RollerEncoder_EVQWGD001, zzkeeb:RotaryEncoder_EVQWGD001, F.Cu at (198.9, 21.5)
- D1, D10, D11, D12, D13, D14, D15, D16, D17, D18, D2, D3, D4, D5, D6, D7, D8, D9: footprint zzkeeb:Diode_1N4148-SOD123-no-label-reversible -> zzkeeb:Diode_1N4148-SOD123; moved to B.Cu
- H1, H2, H3, H4, H5, H6, H7: footprint zzkeeb:Hole_M2-TH -> zzkeeb:Hole_M2-solder-nut-2.5
- J4: moved to B.Cu
- SW1, SW10, SW11, SW12, SW13, SW14, SW15, SW16, SW17, SW18, SW2, SW3, SW4, SW5, SW6, SW7, SW8, SW9: footprint zzkeeb:Switch_KS-miny-reversible-hotswap-south -> zzkeeb:Switch_MXKS-miny-hotswap-south-ks3d
- moved D6 132.4 mm to (170.8, 65.7), turned to 90 degrees
- moved D1 131.4 mm to (167.8, 65.7), turned to 90 degrees
- moved D11 113.3 mm to (167.8, 91.2), turned to 90 degrees
- moved J5 99.4 mm to (233.2, 83.9), turned to 90 degrees
- moved D12 98.6 mm to (170.8, 91.2), turned to 90 degrees
- moved D13 98.3 mm to (170.8, 97.7), turned to 90 degrees
- moved D2 95.6 mm to (167.8, 58.7), turned to 90 degrees
- moved D8 93.2 mm to (167.8, 72.7), turned to 90 degrees
- moved D7 92.2 mm to (164.8, 72.7), turned to 90 degrees
- moved D3 90.7 mm to (164.8, 58.7), turned to 90 degrees
- moved H7 67.1 mm to (199.9, 31.5)
- moved SW38 65.6 mm to (199.9, 21.5), turned to 180 degrees
- moved J6 63.6 mm to (199.9, -3.51)
- moved H1 62.6 mm to (181.4, -20.0)
- moved H2 62.6 mm to (181.4, 21.0)
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Connections:
- J1 pad 2: col5-mcu -> col4-mcu
- J1 pad 20: OFF -> col3-mcu
- J1 pad 31: encA -> OFF
- J1 pad 32: encB -> free2-mcu
- J1 pad 33: unconnected-(J1-107-Pad33) -> free1-mcu
- J1 pad 7: col4-mcu -> encA
- J1 pad 8: col3-mcu -> encB
- J10 pad 12: GND -> free-conn1
- J10 pad 2: col5-conn1 -> col4-conn1
- J10 pad 3: col4-conn1 -> col3-conn1
- J10 pad 4: col3-conn1 -> col2-conn1
- J10 pad 5: col2-conn1 -> col1-conn1
- J10 pad 6: col1-conn1 -> col0-conn1
- J10 pad 7: col0-conn1 -> GND
- J11 pad 12: GND -> free-conn2
- J11 pad 2: col5-conn2 -> col4-conn2
- J11 pad 3: col4-conn2 -> col3-conn2
- J11 pad 4: col3-conn2 -> col2-conn2
- J11 pad 5: col2-conn2 -> col1-conn2
- J11 pad 6: col1-conn2 -> col0-conn2
- J11 pad 7: col0-conn2 -> GND
- J2 pad 12: GND -> free1-mcu
- J2 pad 2: col5-mcu -> col4-mcu
- J2 pad 3: col4-mcu -> col3-mcu
- J2 pad 4: col3-mcu -> col2-mcu
- J2 pad 5: col2-mcu -> col1-mcu
- J2 pad 6: col1-mcu -> col0-mcu
- J2 pad 7: col0-mcu -> GND
- J3 pad 1: GND -> free2-mcu
- J3 pad 10: col4-mcu -> col3-mcu
- J3 pad 11: col5-mcu -> col4-mcu
- J3 pad 6: col0-mcu -> GND
- J3 pad 7: col1-mcu -> col0-mcu
- J3 pad 8: col2-mcu -> col1-mcu
- J3 pad 9: col3-mcu -> col2-mcu
- J4 pad 1: GND -> BAT-left
- J4 pad 10: col4-left -> row1
- J4 pad 11: col5-left -> row0
- J4 pad 12: BAT-left -> unconnected-(J4-Pin_12-Pad12)
- J4 pad 2: row0 -> col4
- J4 pad 3: row1 -> col3
- J4 pad 4: row2 -> col2
- J4 pad 5: row3 -> col1
- J4 pad 6: col0-left -> col0
- J4 pad 7: col1-left -> GND
- J4 pad 8: col2-left -> row3
- J4 pad 9: col3-left -> row2
- J5 pad 1: BAT-left -> unconnected-(J5-Pin_1-Pad1)
- J5 pad 10: row1 -> col8
- J5 pad 11: row0 -> col9
- J5 pad 12: GND -> BAT-right
- J5 pad 2: col5-left -> row7
- J5 pad 3: col4-left -> row6
- J5 pad 4: col3-left -> row5
- J5 pad 5: col2-left -> row4
- J5 pad 6: col1-left -> GND
- J5 pad 7: col0-left -> col5
- J5 pad 8: row3 -> col6
- J5 pad 9: row2 -> col7
- J8 pad 12: GND -> free-conn1
- J8 pad 2: col5-conn1 -> col4-conn1
- J8 pad 3: col4-conn1 -> col3-conn1
- J8 pad 4: col3-conn1 -> col2-conn1
- J8 pad 5: col2-conn1 -> col1-conn1
- J8 pad 6: col1-conn1 -> col0-conn1
- J8 pad 7: col0-conn1 -> GND
- J9 pad 12: GND -> free-conn2
- J9 pad 2: col5-conn2 -> col4-conn2
- J9 pad 3: col4-conn2 -> col3-conn2
- J9 pad 4: col3-conn2 -> col2-conn2
- J9 pad 5: col2-conn2 -> col1-conn2
- J9 pad 6: col1-conn2 -> col0-conn2
- J9 pad 7: col0-conn2 -> GND
- SW1 pad 2: col0-left -> col0
- SW10 pad 2: col4-left -> col4
- SW11 pad 2: col0-left -> col0
- SW12 pad 2: col1-left -> col1
- SW13 pad 2: col2-left -> col2
- SW14 pad 2: col3-left -> col3
- SW15 pad 2: col4-left -> col4
- SW16 pad 2: col2-left -> col2
- SW17 pad 2: col3-left -> col3
- SW18 pad 2: col4-left -> col4
- SW2 pad 2: col1-left -> col1
- SW3 pad 2: col2-left -> col2
- SW4 pad 2: col3-left -> col3
- SW5 pad 2: col4-left -> col4
- SW6 pad 2: col0-left -> col0
- SW7 pad 2: col1-left -> col1
- SW8 pad 2: col2-left -> col2
- SW9 pad 2: col3-left -> col3
Routing:
- net GND: track 143.8 -> 370.3 mm, vias 3 -> 5
- net col2: track 0.00 -> 145.7 mm, vias 0 -> 6
- net col0: track 0.00 -> 143.3 mm
- net col9: track 0.00 -> 138.1 mm, vias 0 -> 3
- net Net-(D23-A): track 0.00 -> 134.2 mm
- net col3: track 0.00 -> 129.3 mm, vias 0 -> 7
- net col7: track 0.00 -> 128.9 mm, vias 0 -> 5
- net Net-(D1-A): track 0.00 -> 121.7 mm
- net col1: track 0.00 -> 119.7 mm, vias 0 -> 4
- net Net-(D28-A): track 0.00 -> 118.2 mm
- net Net-(D33-A): track 0.00 -> 116.7 mm
- net col6: track 0.00 -> 112.1 mm, vias 0 -> 5
- net Net-(D6-A): track 0.00 -> 106.7 mm
- net col4: track 0.00 -> 105.5 mm, vias 0 -> 6
- net Net-(D11-A): track 0.00 -> 103.1 mm
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- removed copper zone on B.Cu, net GND
- removed copper zone on F.Cu, net GND
Other:
- board size 206.4 x 90.7 mm -> 302.4 x 172.7 mm
- board text added: "JLCJLCJLCJLC"
- board text added: "github.com/zzeneg/molekula"
- board text added: "molekula"
- board text added: "v0.1"
- board text removed: "github.com/zzeneg/trio"

Commit message: update pin names
Connections:
- J1 pad 10: row5-mcu -> row6-mcu
- J1 pad 11: row6-mcu -> row5-mcu
- J1 pad 12: row7-mcu -> row4-mcu
- J1 pad 9: row4-mcu -> row7-mcu
- J3 pad 2: row4-mcu -> row7-mcu
- J3 pad 3: row5-mcu -> row6-mcu
- J3 pad 4: row6-mcu -> row5-mcu
- J3 pad 5: row7-mcu -> row4-mcu
Routing:
- net row7-mcu: track 16.0 -> 26.3 mm
- net row4-mcu: track 26.3 -> 16.0 mm
- net row6-mcu: track 19.4 -> 22.9 mm
- net row5-mcu: track 22.9 -> 19.4 mm

Commit message: update case and main pcb
Parts:
- removed U1: RollerEncoder_EVQWGD001, zzkeeb:RotaryEncoder_EVQWGD001
- moved J6 11.5 mm to (199.9, -15.0)
- moved J2 3.50 mm to (195.9, 8.99)
- moved J3 3.50 mm to (203.9, 8.99)
- moved D19 2.76 mm to (234.9, 65.5)
- moved D23 2.76 mm to (231.9, 65.5)
- moved D24 2.76 mm to (228.9, 91.0)
- moved D25 2.76 mm to (234.9, 72.5)
- moved D26 2.76 mm to (231.9, 72.5)
- moved D27 2.76 mm to (228.9, 72.5)
- moved D28 2.76 mm to (228.9, 65.5)
- moved D29 2.76 mm to (234.9, 98.0)
- moved D30 2.76 mm to (231.9, 98.0)
- moved D31 2.76 mm to (228.9, 98.0)
- moved D32 2.76 mm to (234.9, 91.0)
- moved D33 2.76 mm to (231.9, 91.0)
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Routing:
- net MOSI: track 52.8 -> 31.6 mm
- net +3.3V: track 48.1 -> 29.2 mm
- net OFF: track 52.3 -> 37.9 mm
- net CS: track 51.7 -> 37.3 mm, vias 1 -> 0
- net SCK: track 41.5 -> 28.0 mm
- net GND: track 370.3 -> 363.7 mm, vias 5 -> 6
- net encB: track 40.4 -> 35.4 mm
- net BAT-mcu: track 43.0 -> 47.6 mm
- net free1-mcu: track 19.5 -> 23.1 mm
- net encA: track 46.8 -> 43.3 mm
- net row3-mcu: track 15.3 -> 18.8 mm
- net row2-mcu: track 18.8 -> 22.3 mm
- net row1-mcu: track 22.2 -> 25.7 mm
- net row0-mcu: track 25.6 -> 29.1 mm
- net col3-mcu: track 36.2 -> 39.7 mm
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Other:
- board size 302.4 x 172.7 mm -> 301 x 170.2 mm
- board text added: "v0.2"
- board text removed: "JLCJLCJLCJLC"

Commit message: move thumbs to inner side
Parts:
- moved SW34 4.10 mm to (229.1, 124.0)
- moved SW35 4.08 mm to (248.7, 118.8)
- moved SW16 4.00 mm to (130.9, 117.0)
- moved SW17 4.00 mm to (151.1, 118.8)
- moved SW18 4.00 mm to (170.7, 124.0)
- moved SW36 4.00 mm to (268.9, 117.0)
- moved J7 2.12 mm to (169.4, 104.5), turned to 90 degrees
- moved J12 0.71 mm to (230.4, 102.5), turned to -90 degrees
- moved D13 0.50 mm to (170.9, 98.0)
- moved D14 0.50 mm to (167.9, 98.0)
- moved D15 0.50 mm to (164.9, 98.0)
Routing:
- net BAT-left: track 28.8 -> 33.3 mm
- net Net-(D35-A): track 30.4 -> 34.3 mm
- net Net-(D36-A): track 48.3 -> 52.0 mm
- net Net-(D17-A): track 23.5 -> 26.5 mm
- net GND: track 363.7 -> 366.5 mm
- net Net-(D16-A): track 36.0 -> 38.2 mm
- net Net-(D34-A): track 18.2 -> 19.9 mm
- net Net-(D18-A): track 29.7 -> 28.0 mm
- net col4: track 105.5 -> 107.2 mm
- net col5: track 87.1 -> 85.7 mm
- net col7: track 128.9 -> 130.0 mm
- net col6: track 112.1 -> 113.1 mm
- net col2: track 145.7 -> 146.7 mm
- net BAT-right: track 28.5 -> 27.8 mm
- net col3: track 129.3 -> 130.0 mm
Other:
- outline, holes or cut-outs redrawn
- board text added: "v0.3"
- board text removed: "v0.1"

Commit message: pcba version
Parts:
- D1, D10, D11, D12, D13, D14, D15, D16, D17, D18, D19, D2, D20, D21, D22, D23, D24, D25, D26, D27, D28, D29, D3, D30, D31, D32, D33, D34, D35, D36, D4, D5, D6, D7, D8, D9: value D -> C81598
- H1, H2, H3, H4, H5, H6, H7, J10, J6, SW38: moved to B.Cu
- J1, J11, SW37: moved to F.Cu
- J2, J3: value Conn_01x12_Socket -> C479750; moved to B.Cu
- J4, J5: value Conn_01x12_Socket -> C479750
- J8, J9: value Conn_01x12_Socket -> C262499; moved to B.Cu
- SW1, SW10, SW11, SW12, SW13, SW14, SW15, SW19, SW2, SW20, SW21, SW22, SW23, SW24, SW25, SW26, SW27, SW28, SW29, SW3, SW30, SW31, SW32, SW33, SW4, SW5, SW6, SW7, SW8, SW9: footprint zzkeeb:Switch_MXKS-miny-hotswap-south-ks3d -> zzkeeb:Switch_MXKSChoc-miny-hotswap-chocv2-3d
- SW16, SW17, SW18, SW34, SW35, SW36: footprint zzkeeb:Switch_MXKS-miny-hotswap-south-ks3d -> zzkeeb:Switch_KSChoc-miny-hotswap-chocv2-3d
- moved H1 180.8 mm to (314.9, 101.9), turned to 90 degrees
- moved H3 180.8 mm to (84.9, 101.9), turned to -90 degrees
- moved J10 156.1 mm to (297.4, 101.9), turned to 90 degrees
- moved J11 156.1 mm to (102.4, 101.9), turned to 90 degrees
- moved J8 137.0 mm to (283.9, 101.9), turned to 180 degrees
- moved J9 137.0 mm to (115.9, 101.9), turned to 180 degrees
- moved H2 122.9 mm to (273.9, 101.9), turned to 90 degrees
- moved H4 122.9 mm to (125.9, 101.9), turned to -90 degrees
- moved H5 78.5 mm to (214.4, 40.0), turned to 180 degrees
- moved H6 78.5 mm to (185.4, 40.0), turned to 180 degrees
- moved J2 73.4 mm to (203.9, 82.0)
- moved J3 73.4 mm to (195.9, 82.0)
- moved H7 73.0 mm to (199.9, 104.5), turned to 180 degrees
- moved J1 73.0 mm to (199.9, 53.5), turned to 0 degrees
- moved J6 73.0 mm to (199.9, 58.0), turned to 180 degrees
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Connections:
- J9 pad 1: BAT-conn2 -> free-conn2
- J9 pad 10: row1-conn2 -> col3-conn2
- J9 pad 11: row0-conn2 -> col4-conn2
- J9 pad 12: free-conn2 -> BAT-conn2
- J9 pad 2: col4-conn2 -> row0-conn2
- J9 pad 3: col3-conn2 -> row1-conn2
- J9 pad 4: col2-conn2 -> row2-conn2
- J9 pad 5: col1-conn2 -> row3-conn2
- J9 pad 6: col0-conn2 -> GND
- J9 pad 7: GND -> col0-conn2
- J9 pad 8: row3-conn2 -> col1-conn2
- J9 pad 9: row2-conn2 -> col2-conn2
Routing:
- net GND: track 366.5 -> 400.7 mm, vias 6 -> 11
- net col0: track 143.3 -> 161.0 mm, vias 0 -> 4
- net Net-(D18-A): track 28.0 -> 25.5 mm
- net Net-(D17-A): track 26.5 -> 28.5 mm
- net col7: track 130.0 -> 132.0 mm
- net Net-(D23-A): track 134.2 -> 135.4 mm
- net Net-(D28-A): track 118.2 -> 119.1 mm
- net col5: track 85.7 -> 86.4 mm
- net col1: track 119.7 -> 120.3 mm
- added copper zone on B.Cu, net GND
- added copper zone on F.Cu, net GND
Other:
- board size 301 x 170.2 mm -> 276 x 87.2 mm
- board text added: "v0.5"
- board text removed: "v0.2"
- board text removed: "v0.3"
