File: pcb/pcb.kicad_pcb (KiCad board)
At the start: 2 copper layers, 276 x 87.2 mm, 93 parts, among them J1 N!N, J10 Conn_01x12_Socket, J11 Conn_01x12_Socket, J12 Conn_01x02_Socket, J2 C479750, J3 C479750, J4 C479750, J5 C479750, J6 Display_nice-view, J7 Conn_01x02_Socket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

Commit message: small updates
Connections:
- SW37 pad 1: RST -> GND
- SW37 pad 2: GND -> RST
Routing:
- net GND: track 400.7 -> 365.3 mm
- net col4-mcu: track 47.6 -> 51.2 mm
- net RST: track 11.2 -> 14.2 mm
- net BAT-mcu: track 47.6 -> 48.1 mm
Other:
- outline, holes or cut-outs redrawn
