File: pcb/center.kicad_pcb (KiCad board)
At the start: 2 copper layers, 44.6 x 70.5 mm, 17 parts, among them J1 N!N, J10 Conn_01x12_Socket, J11 Conn_01x12_Socket, J2 C479750, J3 C479750, J6 Display_nice-view, J8 C262499, J9 C262499, SW37 SW_Push, SW38 RotaryEncoder_Switch

Commit message: small updates
Connections:
- SW37 pad 1: RST -> GND
- SW37 pad 2: GND -> RST
Routing:
- net GND: track 319.3 -> 282.3 mm
- net col4-mcu: track 47.6 -> 51.2 mm
- net RST: track 11.2 -> 14.2 mm
- net BAT-mcu: track 47.6 -> 48.1 mm
Other:
- outline, holes or cut-outs redrawn
