File: keyboards/Molekula2/pcb.kicad_pcb (KiCad board)
At the start: 2 copper layers, 276 x 87.2 mm, 93 parts, among them J1 N!N, J10 Conn_01x12_Socket, J11 Conn_01x12_Socket, J12 Conn_01x02_Socket, J2 C479750, J3 C479750, J4 C479750, J5 C479750, J6 Display_nice-view, J7 Conn_01x02_Socket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

Commit message: improve combined pcb
Routing:
- net GND: track 365.3 -> 358.6 mm
Other:
- outline, holes or cut-outs redrawn
