File: pcbs/tws-xiao-encoder/tws-xiao-encoder.kicad_pcb (KiCad board)
At the start: 2 copper layers, 30 x 52.5 mm, 9 parts, among them J1 B+, J2 C479750, J5 Conn_01x02_Socket, SW34 SW_SPDT, SW38 RotaryEncoder_Switch, U1 MCU_xiao-ble

Commit message: final choc version
Parts:
- removed J1: B+, Connector_PinHeader_1.00mm:PinHeader_1x01_P1.00mm_Vertical
- added J3: Conn_01x02_Pin, Connector_PinHeader_2.54mm:PinHeader_1x02_P2.54mm_Vertical, F.Cu at (205.4, 61.0)
- added SW37: SW_Push, zzkeeb:Button_SW_SPST_SKQG_WithoutStem, B.Cu at (199.9, 49.0)
Routing:
- net RST: track 0.00 -> 16.4 mm
- net GND: track 45.0 -> 58.7 mm
- net BAT: track 43.3 -> 46.5 mm
- net BAT-mcu: track 23.6 -> 25.9 mm
