File: pcbs/tws-xiao-encoder/tws-xiao-encoder.kicad_sch (KiCad schematic)
At the start: 9 parts, among them J1 Conn_01x01_Pin, J2 C479750, J5 Conn_01x02_Socket, SW34 SW_SPDT, SW38 RotaryEncoder_Switch, U1 MCU_xiao-ble

Commit message: final choc version
Parts:
- removed J1: Conn_01x01_Pin, Connector_PinHeader_1.00mm:PinHeader_1x01_P1.00mm_Vertical, symbol Connector:Conn_01x01_Pin
- added J3: Conn_01x02_Pin, Connector_PinHeader_2.54mm:PinHeader_1x02_P2.54mm_Vertical, symbol Connector:Conn_01x02_Pin
- added SW37: SW_Push, zzkeeb:Button_SW_SPST_SKQG_WithoutStem, symbol Switch:SW_Push
Connections:
- net BAT-mcu: now also J3.1 (Pin_1)
- net GND: now also SW37.1
- new net RST: J3.2 (Pin_2), SW37.2
